Commit message: updated with xacro

File: src/try1/urdf/filev3.xacro (robot description, xacro)
@@ -1,4 +1,4 @@
 <?xml version="1.0"?>
-<robot name="amazingRobot">
+<robot xmlns:xacro="http://www.ros.org/wiki/xacro" name="amazingRobot">
   <material name="blue">
     <color rgba="0 0 0.8 1"/>
@@ -55,13 +55,4 @@
     </visual>
   </link>
-<link name="wheel_left">
-    <visual>
-      <geometry>
-        <cylinder length="0.05" radius="0.2"/>
-      </geometry>
-	<origin rpy="-pi/2 0.0 0.0" xyz="-0.10 0.4 0.0"/>
-      <material name="white"/>
-    </visual>
-  </link>
 <joint name="one" type="continuous">
 <parent link="base"/>
@@ -80,7 +71,21 @@
 <child link="laser_horiz"/>
 </joint>
-<joint name="five" type="fixed">
+<xacro:macro name="xacro_name" params="suffix reflect">
+<link name="wheel_${suffix}">
+    <visual>
+      <geometry>
+        <cylinder length="0.05" radius="0.2"/>
+      </geometry>
+	<origin rpy="-1.57 0.0 0.0" xyz="-0.10 0.4 0.0"/>
+      <material name="white"/>
+    </visual>
+  </link>
+<joint name="five_${suffix}" type="fixed">
 <parent link="base"/>
-<child link="wheel_left"/>
+<child link="wheel_${suffix}"/>
 </joint>
+</xacro:macro>
+<xacro:xacro_name suffix="left" reflect="1" />
+<xacro:xacro_name suffix="right" reflect="-1" />
+<!--<origin xyz="-0.10 ${reflect * 0.4} 0.0" />-->
 </robot>

Commit message: updated cacro

File: src/try1/urdf/filev3.xacro (robot description, xacro)
@@ -18,5 +18,5 @@
   </visual>
 </link>
-<link name="laser_vert_bottom">
+<!--<link name="laser_vert_bottom">
     <visual>
       <geometry>
@@ -26,6 +26,6 @@
       <material name="white"/>
     </visual>
-  </link>
-<link name="laser_vert_top_right">
+  </link>-->
+<!--<link name="laser_vert_top_right">
     <visual>
       <geometry>
@@ -35,6 +35,6 @@
       <material name="white"/>
     </visual>
-  </link>
-<link name="laser_vert_top_left">
+  </link>-->
+<!--<link name="laser_vert_top_left">
     <visual>
       <geometry>
@@ -44,6 +44,6 @@
       <material name="white"/>
     </visual>
-  </link>
-<link name="laser_horiz">
+  </link>-->
+<!--<link name="laser_horiz">
     <visual>
       <parent link="base"/>
@@ -54,21 +54,51 @@
       <material name="white"/>
     </visual>
-  </link>
+  </link>-->
 <joint name="one" type="continuous">
 <parent link="base"/>
 <child link="laser_vert_bottom"/>
 </joint>
-<joint name="two" type="continuous">
+<!--<joint name="two" type="continuous">
 <parent link="base"/>
 <child link="laser_vert_top_right"/>
-</joint>
-<joint name="three" type="continuous">
+</joint>-->
+<!--<joint name="three" type="continuous">
 <parent link="base"/>
 <child link="laser_vert_top_left"/>
-</joint>
-<joint name="four" type="continuous">
+</joint>-->
+<!--<joint name="four" type="continuous">
 <parent link="base"/>
 <child link="laser_horiz"/>
+</joint>-->
+<!--<xacro:macro name="xacro_name2" params="suffix reflect">-->
+<link name="wheel_center">
+    <visual>
+      <geometry>
+        <cylinder length="0.05" radius="0.15"/>
+      </geometry>
+		<origin xyz="-0.10 0.0 0.0" rpy="-1.57 0.0 0.0"/>
+	<!--<origin rpy="-1.57 0.0 0.0" xyz="-0.10 0.4 0.0"/>-->
+      <material name="white"/>
+    </visual>
+  </link>
+<joint name="six" type="continuous">
+<parent link="base"/>
+<child link="wheel_center"/>
 </joint>
+<!--</xacro:macro>
+<xacro:xacro_name suffix="center" reflect="1" />-->
+<xacro:include filename="$(find velodyne_description)/urdf/VLP-16.urdf.xacro"/>
+<VLP-16 parent="base" name="laser_horiz" topic="laser_horiz/packets" hz="10"
+samples="440" gpu="false">
+<origin xyz="0.2325416305773505 -0.0001380069427607134 1.920122926231907" rpy="-0.0012068 0.114646 -0.0015308" />
+</VLP-16>
+<xacro:include filename="$(find gazebo_plugins)/test/multi_robot_scenario/xacro/laser/hokuyo.xacro"/>
+<xacro:laser name="laser_vert_bottom" parent="base" xyz="0.3157894464801903
+-0.002068548615034871 0.5099999434059285" rpy="3.1354753 -1.3045001 0.0024658"
+meshes="package://gazebo_plugins/test/multi_robot_scenario/meshes/laser" />
+<xacro:laser name="laser_vert_right" parent="base" xyz="0.2978 -0.1450 1.8451" rpy="-1.1760 0.6313 -1.9377"
+meshes="package://gazebo_plugins/test/multi_robot_scenario/meshes/laser" />
+<xacro:laser name="laser_vert_left" parent="base" rpy="1.1780 0.6198 1.9560" xyz="0.2997 0.1531 1.8443"
+meshes="package://gazebo_plugins/test/multi_robot_scenario/meshes/laser" />
 <xacro:macro name="xacro_name" params="suffix reflect">
 <link name="wheel_${suffix}">
@@ -77,9 +107,10 @@
         <cylinder length="0.05" radius="0.2"/>
       </geometry>
-	<origin rpy="-1.57 0.0 0.0" xyz="-0.10 0.4 0.0"/>
+		<origin xyz="-0.10 ${reflect * 0.4} 0.0" rpy="-1.57 0.0 0.0"/>
+	<!--<origin rpy="-1.57 0.0 0.0" xyz="-0.10 0.4 0.0"/>-->
       <material name="white"/>
     </visual>
   </link>
-<joint name="five_${suffix}" type="fixed">
+<joint name="five_${suffix}" type="continuous">
 <parent link="base"/>
 <child link="wheel_${suffix}"/>

File: src/try1/urdf/new.urdf (robot description, URDF)
Before this commit: robot amazingRobot, 7 links, 6 joints
Links:
- removed link laser_vert_top_left
- removed link laser_vert_top_right
- added link laser_horiz_base_link, mass 0.83; collision cylinder length=0.0717 radius=0.0516; visual mesh filename=package://velodyne_description/meshes/VLP16_base_1.dae
- added link laser_vert_left, mass 1e-5; collision box size=0.1 0.1 0.1; visual mesh filename=package://gazebo_plugins/test/multi_robot_scenario/meshes/l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
- added link laser_vert_right, mass 1e-5; collision box size=0.1 0.1 0.1; visual mesh filename=package://gazebo_plugins/test/multi_robot_scenario/meshes/l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
- added link wheel_center; visual cylinder length=0.05 radius=0.15
- link laser_horiz: mass None -> 0.01; geometry visual mesh filename=package://velodyne_description/meshes/VLP16_scan.dae
- link laser_vert_bottom: mass None -> 1e-5; geometry collision box size=0.1 0.1 0.1; visual mesh filename=package://gazebo_plugins/test/multi_robot_scenario/meshes/l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
Joints:
- removed joint four
- removed joint three
- removed joint two
- added joint base_laser_vert_bottom_joint: type fixed, parent base, child laser_vert_bottom, origin xyz=0.3157894464801903 -0.002068548615034871 0.5099999434059285 rpy=3.1354753 -1.3045001 0.0024658, axis 0 0 1
- added joint base_laser_vert_left_joint: type fixed, parent base, child laser_vert_left, origin xyz=0.2997 0.1531 1.8443 rpy=1.1780 0.6198 1.9560, axis 0 0 1
- added joint base_laser_vert_right_joint: type fixed, parent base, child laser_vert_right, origin xyz=0.2978 -0.1450 1.8451 rpy=-1.1760 0.6313 -1.9377, axis 0 0 1
- added joint laser_horiz_base_mount_joint: type fixed, parent base, child laser_horiz_base_link, origin xyz=0.2325416305773505 -0.0001380069427607134 1.920122926231907 rpy=-0.0012068 0.114646 -0.0015308
- added joint laser_horiz_base_scan_joint: type fixed, parent laser_horiz_base_link, child laser_horiz, origin xyz=0 0 0.0377 rpy=0 0 0
- added joint six: type continuous, parent base, child wheel_center
- joint five_left: type fixed -> continuous
- joint five_right: type fixed -> continuous
